File: hardware/board/environment_sensor/environment_sensor.kicad_pcb (KiCad board)
At the start: 4 copper layers, 28 x 28 mm, 47 parts, among them J2 AudioJack3, J3 USB_C_Receptacle_USB2.0, SW1 SW_Push, U1 TPD2EUSB30, U2 LP2985-3.3, U3 RP2040, U4 W25Q16JVUXIQ, U5 BME688, X1 ECS-TXO-2016

Commit message: draft v0.1 pcb
Parts:
- moved C2 0.22 mm to (138.7, 96.9)
- moved C15 0.22 mm to (140.9, 96.9)
- moved C6 0.20 mm to (139.8, 96.9)
- moved C16 0.20 mm to (143.1, 91.7)
- moved X1 0.14 mm to (136.9, 97.3)
- moved C24 0.10 mm to (144.0, 98.6)
- moved C25 0.10 mm to (144.6, 99.6)
- moved C26 0.10 mm to (144.6, 100.6)
- moved C12 0.10 mm to (143.9, 85.0)
Connections:
- U3 pad 2: /Harp Core RP2040 + USB/UART0_TXD -> unconnected-(U3-GPIO0-Pad2)
- U3 pad 24: /Harp Core RP2040 + USB/SWCLK -> unconnected-(U3-SWCLK-Pad24)
- U3 pad 25: /Harp Core RP2040 + USB/SWDIO -> unconnected-(U3-SWD-Pad25)
- U3 pad 27: unconnected-(U3-GPIO16-Pad27) -> /Harp Core RP2040 + USB/POCI
- U3 pad 29: unconnected-(U3-GPIO18-Pad29) -> /Harp Core RP2040 + USB/SCK
- U3 pad 3: /Harp Core RP2040 + USB/UART0_RXD -> unconnected-(U3-GPIO1-Pad3)
- U3 pad 30: unconnected-(U3-GPIO19-Pad30) -> /Harp Core RP2040 + USB/PICO
- U3 pad 31: unconnected-(U3-GPIO20-Pad31) -> /Harp Core RP2040 + USB/CS
- U3 pad 4: /Harp Core RP2040 + USB/SCK -> unconnected-(U3-GPIO2-Pad4)
- U3 pad 5: /Harp Core RP2040 + USB/PICO -> unconnected-(U3-GPIO3-Pad5)
- U3 pad 6: /Harp Core RP2040 + USB/POCI -> unconnected-(U3-GPIO4-Pad6)
- U3 pad 8: /Harp Core RP2040 + USB/CS -> unconnected-(U3-GPIO6-Pad8)
Routing:
- net /Harp Core RP2040 + USB/PICO: track 16.9 -> 3.70 mm
- net /Harp Core RP2040 + USB/SCK: track 13.9 -> 2.74 mm
- net /Harp Core RP2040 + USB/POCI: track 15.2 -> 5.03 mm
- net GND: track 26.3 -> 32.6 mm, vias 24 -> 26
- net /Harp Core RP2040 + USB/CS: track 0.00 -> 4.87 mm, vias 0 -> 1
- net /Harp Core RP2040 + USB/D+: track 24.9 -> 22.2 mm
- net /Harp Core RP2040 + USB/D-: track 25.2 -> 23.3 mm
- net +3V3: track 45.8 -> 46.3 mm, vias 12 -> 16
Other:
- outline, holes or cut-outs redrawn
- board text added: "1"
- board text added: "BME688"
- board text added: "Expose sensor from enclosure ↓"
- board text added: "V0.1.0"
- board text added: "Vasquez, Sept 6, 2023"

Commit message: update 3.5mm connector orientation and 3d models
Parts:
- moved C10 8.96 mm to (148.2, 98.2), turned to 90 degrees
- moved D1 8.84 mm to (147.2, 98.2), turned to -90 degrees
- moved C24 0.20 mm to (143.8, 98.6)
- moved C25 0.20 mm to (144.4, 99.6)
- moved C26 0.20 mm to (144.4, 100.6)
- turned J2 to 180 degrees
Routing:
- net GND: track 32.6 -> 36.3 mm, vias 26 -> 29
- net /Harp Core RP2040 + USB/HARP_CLK_SYNC: track 32.4 -> 35.6 mm
- net +3V3: track 46.3 -> 43.5 mm, vias 16 -> 18
Other:
- board text added: "V0.1.1"
- board text added: "Vasquez, Oct 23, 2023"
- board text removed: "V0.1.0"
- board text removed: "Vasquez, Sept 6, 2023"

Commit message: bugfix starting bytes written
Parts:
- added REF**: MountingHole_2.2mm_M2_DIN965, MountingHole:MountingHole_2.2mm_M2_DIN965, F.Cu at (160.0, 84.0)
- added REF**: MountingHole_2.2mm_M2_DIN965, MountingHole:MountingHole_2.2mm_M2_DIN965, F.Cu at (128.0, 108.0)
- added REF**: MountingHole_2.2mm_M2_DIN965, MountingHole:MountingHole_2.2mm_M2_DIN965, F.Cu at (160.0, 108.0)
- added REF**: MountingHole_2.2mm_M2_DIN965, MountingHole:MountingHole_2.2mm_M2_DIN965, F.Cu at (128.0, 84.0)
Other:
- board size 28 x 28 mm -> 36 x 28 mm
- board text added: "Nov 8, 2023"
- board text added: "Sonya Vasquez"
- board text removed: "Vasquez, Oct 23, 2023"
Changed lines of the file:
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@@
     )
     (pad_to_mask_clearance 0)
-    (aux_axis_origin 130 110)
+    (aux_axis_origin 126 110)
     (pcbplotparams
       (layerselection 0x00010fc_ffffffff)
@@
     )
   )
+  (footprint "MountingHole:MountingHole_2.2mm_M2_DIN965" (layer "F.Cu")
+    (at 160 84)
+    (descr "Mounting Hole 2.2mm, no annular, M2, DIN965")
+    (tags "mounting hole 2.2mm no annular m2 din965")
+    (attr exclude_from_pos_files exclude_from_bom)
+    (fp_text reference "REF**" (at 0 -2.9) (layer "F.SilkS") hide
+        (effects (font (size 1 1) (thickness 0.15)))
+    )
+    (fp_text value "MountingHole_2.2mm_M2_DIN965" (at 0 2.9) (layer "F.Fab") hide
+        (effects (font (size 1 1) (thickness 0.15)))
+    )
+    (fp_text user "${REFERENCE}" (at 0 0) (layer "F.Fab") hide
+        (effects (font (size 1 1) (thickness 0.15)))
+    )
+    (fp_circle (center 0 0) (end 1.9 0)
+      (stroke (width 0.15) (type solid)) (fill none) (layer "Cmts.User"))
+    (fp_circle (center 0 0) (end 2.15 0)
+      (stroke (width 0.05) (type solid)) (fill none) (layer "F.CrtYd"))
+    (pad "" np_thru_hole circle (at 0 0) (size 2.2 2.2) (drill 2.2) (layers "*.Mask" "F.Cu" "In1.Cu" "In2.Cu" "B.Cu"))
+  )
   (footprint "Fiducial:Fiducial_0.5mm_Mask1mm" (layer "F.Cu")
     (at 130.8 82.8)
@@
     )
   )
+  (footprint "MountingHole:MountingHole_2.2mm_M2_DIN965" (layer "F.Cu")
+    (at 128 108)
+    (descr "Mounting Hole 2.2mm, no annular, M2, DIN965")
+    (tags "mounting hole 2.2mm no annular m2 din965")
+    (attr exclude_from_pos_files exclude_from_bom)
+    (fp_text reference "REF**" (at 0 -2.9) (layer "F.SilkS") hide
+        (effects (font (size 1 1) (thickness 0.15)))
+    )
+    (fp_text value "MountingHole_2.2mm_M2_DIN965" (at 0 2.9) (layer "F.Fab") hide
+        (effects (font (size 1 1) (thickness 0.15)))
+    )
+    (fp_text user "${REFERENCE}" (at 0 0) (layer "F.Fab") hide
+        (effects (font (size 1 1) (thickness 0.15)))
+    )
+    (fp_circle (center 0 0) (end 1.9 0)
+      (stroke (width 0.15) (type solid)) (fill none) (layer "Cmts.User"))
+    (fp_circle (center 0 0) (end 2.15 0)
+      (stroke (width 0.05) (type solid)) (fill none) (layer "F.CrtYd"))
+    (pad "" np_thru_hole circle (at 0 0) (size 2.2 2.2) (drill 2.2) (layers "*.Mask" "F.Cu" "In1.Cu" "In2.Cu" "B.Cu"))
+  )
   (footprint "Capacitor_SMD:C_0402_1005Metric" (layer "F.Cu")
     (at 144.4 100.6 180)
@@
     )
   )
+  (footprint "MountingHole:MountingHole_2.2mm_M2_DIN965" (layer "F.Cu")
+    (at 160 108)
+    (descr "Mounting Hole 2.2mm, no annular, M2, DIN965")
+    (tags "mounting hole 2.2mm no annular m2 din965")
+    (attr exclude_from_pos_files exclude_from_bom)
+    (fp_text reference "REF**" (at 0 -2.9) (layer "F.SilkS") hide
+        (effects (font (size 1 1) (thickness 0.15)))
+    )
+    (fp_text value "MountingHole_2.2mm_M2_DIN965" (at 0 2.9) (layer "F.Fab") hide
+        (effects (font (size 1 1) (thickness 0.15)))
+    )
+    (fp_text user "${REFERENCE}" (at 0 0) (layer "F.Fab") hide
+        (effects (font (size 1 1) (thickness 0.15)))
+    )
+    (fp_circle (center 0 0) (end 1.9 0)
+      (stroke (width 0.15) (type solid)) (fill none) (layer "Cmts.User"))
+    (fp_circle (center 0 0) (end 2.15 0)
+      (stroke (width 0.05) (type solid)) (fill none) (layer "F.CrtYd"))
+    (pad "" np_thru_hole circle (at 0 0) (size 2.2 2.2) (drill 2.2) (layers "*.Mask" "F.Cu" "In1.Cu" "In2.Cu" "B.Cu"))
+  )
   (footprint "Connector_USB:USB_C_Receptacle_JAE_DX07S016JA1R1500" (layer "F.Cu")
     (at 138.6 106.2)
@@
     )
   )
+  (footprint "MountingHole:MountingHole_2.2mm_M2_DIN965" (layer "F.Cu")
+    (at 128 84)
+    (descr "Mounting Hole 2.2mm, no annular, M2, DIN965")
+    (tags "mounting hole 2.2mm no annular m2 din965")
+    (attr exclude_from_pos_files exclude_from_bom)
+    (fp_text reference "REF**" (at 0 -2.9) (layer "F.SilkS") hide
+        (effects (font (size 1 1) (thickness 0.15)))
+    )
+    (fp_text value "MountingHole_2.2mm_M2_DIN965" (at 0 2.9) (layer "F.Fab") hide
+        (effects (font (size 1 1) (thickness 0.15)))
+    )
+    (fp_text user "${REFERENCE}" (at 0 0) (layer "F.Fab") hide
+        (effects (font (size 1 1) (thickness 0.15)))
+    )
+    (fp_circle (center 0 0) (end 1.9 0)
+      (stroke (width 0.15) (type solid)) (fill none) (layer "Cmts.User"))
+    (fp_circle (center 0 0) (end 2.15 0)
+      (stroke (width 0.05) (type solid)) (fill none) (layer "F.CrtYd"))
+    (pad "" np_thru_hole circle (at 0 0) (size 2.2 2.2) (drill 2.2) (layers "*.Cu" "*.Mask"))
+  )
   (footprint "Package_LGA:Bosch_LGA-8_3x3mm_P0.8mm_ClockwisePinNumbering" (layer "B.Cu")
     (at 144 96 180)
@@
     )
   )
-  (gr_rect (start 130 82) (end 158 110)
+  (gr_rect (start 126 82) (end 162 110)
     (stroke (width 0.1) (type default)) (fill none) (layer "Cmts.User"))
-  (gr_line (start 157.2 82) (end 130.8 82)
+  (gr_line (start 160 82) (end 128 82)
     (stroke (width 0.1) (type default)) (layer "Edge.Cuts"))
-  (gr_arc (start 130.8 110) (mid 130.234315 109.765685) (end 130 109.2)
+  (gr_arc (start 128 110) (mid 126.585786 109.414214) (end 126 108)
     (stroke (width 0.1) (type default)) (layer "Edge.Cuts"))
-  (gr_line (start 158 109.2) (end 158 82.8)
+  (gr_line (start 162 108) (end 162 84)
     (stroke (width 0.1) (type default)) (layer "Edge.Cuts"))
-  (gr_arc (start 158 109.2) (mid 157.765685 109.765685) (end 157.2 110)
+  (gr_arc (start 162 108) (mid 161.414214 109.414214) (end 160 110)
     (stroke (width 0.1) (type default)) (layer "Edge.Cuts"))
-  (gr_arc (start 157.2 82) (mid 157.765685 82.234315) (end 158 82.8)
+  (gr_arc (start 160 82) (mid 161.414214 82.585786) (end 162 84)
     (stroke (width 0.1) (type default)) (layer "Edge.Cuts"))
-  (gr_line (start 130 82.8) (end 130 109.2)
+  (gr_line (start 126 84) (end 126 108)
     (stroke (width 0.1) (type default)) (layer "Edge.Cuts"))
-  (gr_arc (start 130 82.8) (mid 130.234315 82.234315) (end 130.8 82)
+  (gr_arc (start 126 84) (mid 126.585786 82.585786) (end 128 82)
     (stroke (width 0.1) (type default)) (layer "Edge.Cuts"))
-  (gr_line (start 130.8 110) (end 157.2 110)
+  (gr_line (start 128 110) (end 160 110)
     (stroke (width 0.1) (type default)) (layer "Edge.Cuts"))
   (gr_text "Expose sensor \nfrom enclosure ↓" (at 156.9 93.8) (layer "B.SilkS")
@@
     (effects (font (size 1 1) (thickness 0.13)) (justify left bottom mirror))
   )
-  (gr_text "Vasquez,\nOct 23, 2023" (at 157.7 109.4) (layer "B.SilkS")
-    (effects (font (size 1 1) (thickness 0.13)) (justify left bottom mirror))
+  (gr_text "Harp\nEnvironment\nSensor" (at 157 89.5) (layer "B.SilkS")
+    (effects (font (size 1.4 1.4) (thickness 0.25) bold) (justify left bottom mirror))
   )
-  (gr_text "Harp\nEnvironment\nSensor" (at 157.6 90.3) (layer "F.SilkS")
+  (gr_text "Harp\nEnvironment\nSensor" (at 160.5 92) (layer "F.SilkS")
     (effects (font (size 1.4 1.4) (thickness 0.25) bold) (justify right bottom))
   )
+  (gr_text "Nov 8, 2023" (at 159.5 105.5 90) (layer "F.SilkS")
+    (effects (font (size 1 1) (thickness 0.13)) (justify left bottom))
+  )
+  (gr_text "Sonya Vasquez" (at 161 105.5 90) (layer "F.Mask")
+    (effects (font (size 1 1) (thickness 0.13)) (justify left bottom))
+  )
   (segment (start 136.25 103.65) (end 136.25 103.15) (width 0.25) (layer "F.Cu") (net 1))
   (segment (start 140.95 103.15) (end 140.95 103.65) (width 0.25) (layer "F.Cu") (net 1))
@@
   (via (at 131.8 91.4) (size 0.4572) (drill 0.254) (layers "F.Cu" "B.Cu") (net 11))
   (via (at 155.7 97.8) (size 0.4572) (drill 0.254) (layers "F.Cu" "B.Cu") (net 11))
-  (segment (start 132.0786 95.2786) (end 137.4 100.6) (width 0.1524) (layer "B.Cu") (net 11))
-  (segment (start 152.9 100.6) (end 155.7 97.8) (width 0.1524) (layer "B.Cu") (net 11))
-  (segment (start 137.4 100.6) (end 152.9 100.6) (width 0.1524) (layer "B.Cu") (net 11))
+  (segment (start 132.0786 95.2786) (end 137.6 100.8) (width 0.1524) (layer "B.Cu") (net 11))
+  (segment (start 152.7 100.8) (end 155.7 97.8) (width 0.1524) (layer "B.Cu") (net 11))
+  (segment (start 137.6 100.8) (end 152.7 100.8) (width 0.1524) (layer "B.Cu") (net 11))
   (segment (start 131.8 91.4) (end 132.0786 91.6786) (width 0.1524) (layer "B.Cu") (net 11))
   (segment (start 132.0786 91.6786) (end 132.0786 95.2786) (width 0.1524) (layer "B.Cu") (net 11))
@@
     (polygon
       (pts
-        (xy 130 110)
-        (xy 158 110)
-        (xy 158 82)
-        (xy 130 82)
+        (xy 126 110)
+        (xy 162 110)
+        (xy 162 82)
+        (xy 126 82)
       )
     )
@@
     (polygon
       (pts
-        (xy 130 110)
-        (xy 158 110)
-        (xy 158 82)
-        (xy 130 82)
+        (xy 126 110)
+        (xy 162 110)
+        (xy 162 82)
+        (xy 126 82)
       )
     )
