File: hardware/board/environment_sensor/environment_sensor.kicad_pcb (KiCad board)
At the start: 4 copper layers, 39.9 x 28 mm, 56 parts, among them J2 AudioJack3, J3 USB_C_Receptacle_USB2.0, SW1 SW_Push, U1 TPD2EUSB30, U3 RP2040, U4 W25Q16JVUXIQ, U5 BME688, U6 rt6150b-33gqw, X1 ECS-TXO-2016

Commit message: update CUI -> Same Sky
Parts:
- J2: footprint Connector_Audio:Jack_3.5mm_CUI_SJ-3523-SMT_Horizontal -> Connector_Audio:Jack_3.5mm_CUI_SJ-3524-SMT_Horizontal
- L2: value L -> 2.2uH
- moved D2 0.25 mm to (136.4, 101.6)
- moved R2 0.25 mm to (137.4, 101.6)
Other:
- board text added: "V0.2.0"
- board text removed: "V0.1.1"
