File: hardware/board/environment_sensor/environment_sensor.kicad_sch (KiCad schematic)
At the start: 4 parts, among them U5 BME688

Commit message: draft v0.1 pcb
Parts:
- U5: Link (none) -> https://www.digikey.com/en/products/detail/bosch-sensortec/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
Changed lines of the file:
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@@
+      (effects (font (size 1.27 1.27)) hide)
+    )
+    (property "Link" "https://www.digikey.com/en/products/detail/bosch-sensortec/BME688/13681261" (at 114.3 76.2 0)
       (effects (font (size 1.27 1.27)) hide)
     )

Commit message: update 3.5mm connector orientation and 3d models
Other:
- note added: "BME688 in SPI mode."
Changed lines of the file:
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@@
+    (effects (font (size 1.27 1.27)) (justify left bottom))
+  )
+  (text "BME688 in SPI mode." (at 103.505 106.045 0)
     (effects (font (size 1.27 1.27)) (justify left bottom))
   )

Commit message: update pcb with thermal considerations
Parts:
- renumbered C13 to C24, C13 to C25, C11 to C26
